File: ancuk.kicad_pcb (KiCad board)
At the start: 2 copper layers, 14 parts, among them J1 GSR_Pads, M1 Vibration_Motor, Q1 2N2222, U1 XIAO_ESP32C3, U2 MAX30102_Breakout, U3 OLED_0.42in, U4 MCP6002

Commit message: cok1
Parts:
- moved U2 3.88 mm to (140.0, 51.8)
- moved BT1 3.80 mm to (120.0, 75.7)
- moved U1 3.68 mm to (119.4, 71.1)
- moved U3 1.95 mm to (150.0, 53.0)
Routing:
- net SCL: track 5.64 -> 51.8 mm
- net SDA: track 5.64 -> 49.7 mm, vias 0 -> 1
- net GSR_OUT: track 0.00 -> 32.4 mm, vias 0 -> 2
- net INT: track 0.00 -> 28.1 mm
- net GND: track 40.2 -> 61.6 mm
- net +3V3: track 28.8 -> 48.6 mm, vias 0 -> 2
- net Net-(U1-D3/A3): track 27.2 -> 31.2 mm
- net /BAT+: track 4.59 -> 8.38 mm

Commit message: tolong aku
Parts:
- removed U2: MAX30102_Breakout, Connector_PinHeader_2.54mm:PinHeader_1x05_P2.54mm_Vertical
- added MAX1: MAX 30102, Connector_PinHeader_2.54mm:PinHeader_1x07_P2.54mm_Vertical, F.Cu at (139.8, 49.8)
- J1: footprint TestPoint:TestPoint_Pad_D3.0mm -> Connector_PinHeader_2.54mm:PinHeader_1x02_P2.54mm_Vertical
- M1: footprint TestPoint:TestPoint_Pad_D2.0mm -> Connector_PinHeader_2.54mm:PinHeader_1x02_P2.54mm_Vertical
- TP1: footprint Connector_PinHeader_2.54mm:PinHeader_1x02_P2.54mm_Vertical -> Connector_PinHeader_2.54mm:PinHeader_1x01_P2.54mm_Vertical
- moved J1 1.12 mm to (143.0, 77.0)
- renumbered U3 to OLED1
Connections:
- BT1 pad 2: unconnected-(BT1---Pad2) -> +3V3
- U1 pad 10: unconnected-(U1-GND-Pad10) -> +3V3
- U1 pad 9: unconnected-(U1-5V-Pad9) -> /BAT+
Routing:
- net +3V3: track 48.6 -> 91.4 mm, vias 2 -> 7
- net /BAT+: track 8.38 -> 35.2 mm, vias 0 -> 1
- net (no net): track 17.5 -> 0.00 mm, vias 1 -> 0
- net Net-(D1-A): track 11.1 -> 20.7 mm
- net Net-(J1-Pin_2): track 0.00 -> 8.03 mm, vias 0 -> 1
- net GND: track 61.6 -> 68.5 mm
- net SDA: track 49.7 -> 51.9 mm
- net INT: track 28.1 -> 26.9 mm
- net Net-(U1-D3/A3): track 31.2 -> 32.0 mm, vias 0 -> 2
- net SCL: track 51.8 -> 51.2 mm
Other:
- board outline added: 36 x 35 mm
