File: lomba.kicad_sch (KiCad schematic)
At the start: 13 parts, among them J1 GSR_Pads, M1 Vibration_Motor, Q1 2N2222, U1 XIAO_ESP32C3, U4 MCP6002

Commit message: tolong aku
Parts:
- removed MAX1: MAX 30102, Connector_PinHeader_2.54mm:PinHeader_1x07_P2.54mm_Vertical, symbol Connector_Generic:Conn_01x07
- added TP1: PAD_BAT_PLUS, Connector_PinHeader_2.54mm:PinHeader_1x02_P2.54mm_Vertical, symbol Connector:TestPoint
- added U2: MAX30102_Breakout, Connector_PinHeader_2.54mm:PinHeader_1x05_P2.54mm_Vertical, symbol Connector_Generic:Conn_01x05
- J1: footprint Connector_PinHeader_2.54mm:PinHeader_1x02_P2.54mm_Vertical -> TestPoint:TestPoint_Pad_D3.0mm
- M1: footprint Connector_PinHeader_2.54mm:PinHeader_1x02_P2.54mm_Vertical -> TestPoint:TestPoint_Pad_D2.0mm
- renumbered OLED1 to U3
Connections:
- net +3V3: now also U2.1 (Pin_1); no longer BT1.2 (-), U1.10 (GND)
- net BAT+: now also TP1.1; no longer U1.9 (5V)
- net GND: now also U2.5 (Pin_5)
- net INT: now also U2.4 (Pin_4)
- net SCL: now also U2.2 (Pin_2)
- net SDA: now also U2.3 (Pin_3)
